File: mcu.kicad_sch (KiCad schematic)
At the start: 36 parts, among them J2 USB C, J3 DBG, J4 5V IN, J6 Aux, Q1 PMV65XP, SW1 RESET, U3 DSC61XX, U4 STM32L432KCUx, U5 MCP2562FD

Commit message: pcb: change oscillator footprint, add board id pad and move board name on back silkscreen
Parts:
- U3: footprint Package_LGA:VLGA-4_2x2.5mm_P1.65mm -> Crystal:Crystal_SMD_3225-4Pin_3.2x2.5mm
Changed lines of the file:
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@@
     (property "Reference" "U3" (id 0) (at 26.67 54.61 0))
     (property "Value" "DSC61XX" (id 1) (at 26.67 57.15 0))
-    (property "Footprint" "Package_LGA:VLGA-4_2x2.5mm_P1.65mm" (id 2) (at 26.67 63.5 0)
+    (property "Footprint" "Crystal:Crystal_SMD_3225-4Pin_3.2x2.5mm" (id 2) (at 26.67 63.5 0)
       (effects (font (size 1.27 1.27)) hide)
     )
